File: Hardware/SparkFun RTK Express.brd (EAGLE design)
At the start: 68.2 x 110.1 mm, 166 parts, among them J13 Internal, J16 microSD, J17 Qwiic Right Angle, J3 USB Female Type C Connector, J4 External, J5 USB Female Type C Connector, Q1 SIL2308-TP, Q2 MBT3904DW1T1, U1 74HC4052D, U10 MCP73833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

Commit message: v14 - Remove ground plane from around accelerometer
Parts:
- removed U$18: (no value), output:V130
- added U$12: (no value), output:V140
Routing:
- net GND: track 18.1 -> 37.5 mm
- net 3.3V: track 317.2 -> 329.2 mm, vias 6 -> 8
Other:
- board text added: "JLC7628 Impedance controlled"
